File: PCB/ifidget.sch (KiCad schematic (older format))
At the start: 57 parts, among them P1 USB_OTG, P17 DBG_CONN, P2 BatteryHolder, P3 BatteryHolder, P4 BatteryHolder, Q1 Q_PMOS_DSG, SW2 SW_PUSH, SW3 SW_PUSH, SW4 SW_PUSH, U1 74AHC1G125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

Commit message: updates
Parts:
- removed D6: RX, project_footprints:Led_0603, symbol Led_Small
- removed D7: TX, project_footprints:Led_0603, symbol Led_Small
- removed R13, R14: 1k, project_footprints:R_0402_Hand, symbol R
- added C13: 1uF, project_footprints:C_0402_Hand, symbol C_Small
- added R18, R19, R20, R21, R22, R23: 10k, project_footprints:R_0402_Hand, symbol R
- added U6, U7: TLE4946-2K, idlehands_footprints:SOT23, symbol TLE4946-2K
- C9: Digikey Part No. 587-1059-1-ND -> 1276-1469-1-ND
- D1: Digikey Part No. (none) -> 497-3381-1-ND
- D10, D11, D2, D3, D4, D5, D8, D9: Digikey Part No. (none) -> 160-1436-1-ND
- U4: Digikey Part No. (none) -> 1727-3327-1-ND
- U5: Digikey Part No. (none) -> MCP73831T-2ACI/OTCT-ND
Connections:
- net labels added: HALL1, HALL2
- wire segments 204 -> 230
Other:
- moved on the sheet: SW2, SW3

Commit message: fixes to power and listed issues
Parts:
- removed R22, R23: 10k, project_footprints:R_0402_Hand, symbol R
- added D6: CHRG, idlehands_footprints:Led_0603, symbol LED
- added Q2: 2N7002, TO_SOT_Packages_SMD:SOT-23, symbol 2N7002
- added R13: 100k, project_footprints:R_0402_Hand, symbol R_Small
- added R14: 1K, project_footprints:R_0402_Hand, symbol R
Connections:
- net labels added: HALLSW
- wire segments 230 -> 237
Other:
- moved on the sheet: R16, R17
Changed lines of the file:
@@
 L R R16
 U 1 1 5914E516
-P 6100 9950
-F 0 "R16" V 6180 9950 50  0000 C CNN
-F 1 "10k" V 6100 9950 50  0000 C CNN
-F 2 "project_footprints:R_0402_Hand" V 6030 9950 30  0001 C CNN
-F 3 "" H 6100 9950 30  0000 C CNN
-F 4 "311-10KJRCT-ND" V 6100 9950 60  0001 C CNN "Digikey Part No."
-	1    6100 9950
+P 5250 9050
+F 0 "R16" V 5330 9050 50  0000 C CNN
+F 1 "10k" V 5250 9050 50  0000 C CNN
+F 2 "project_footprints:R_0402_Hand" V 5180 9050 30  0001 C CNN
+F 3 "" H 5250 9050 30  0000 C CNN
+F 4 "311-10KJRCT-ND" V 5250 9050 60  0001 C CNN "Digikey Part No."
+	1    5250 9050
 	-1   0    0    1
 $EndComp
@@
 L R R17
 U 1 1 5914E5DA
-P 6100 10400
-F 0 "R17" V 6180 10400 50  0000 C CNN
-F 1 "20k" V 6100 10400 50  0000 C CNN
-F 2 "project_footprints:R_0402_Hand" V 6030 10400 30  0001 C CNN
-F 3 "" H 6100 10400 30  0000 C CNN
-F 4 "311-20KJRCT-ND" V 6100 10400 60  0001 C CNN "Digikey Part No."
-	1    6100 10400
+P 5250 9500
+F 0 "R17" V 5330 9500 50  0000 C CNN
+F 1 "20k" V 5250 9500 50  0000 C CNN
+F 2 "project_footprints:R_0402_Hand" V 5180 9500 30  0001 C CNN
+F 3 "" H 5250 9500 30  0000 C CNN
+F 4 "311-20KJRCT-ND" V 5250 9500 60  0001 C CNN "Digikey Part No."
+	1    5250 9500
 	-1   0    0    1
 $EndComp
-Text GLabel 6250 10200 2    60   Input ~ 0
+Text GLabel 5400 9300 2    60   Input ~ 0
 STAT
 $Comp
 L GND #PWR032
 U 1 1 5914EC58
-P 6100 10700
-F 0 "#PWR032" H 6100 10450 50  0001 C CNN
-F 1 "GND" H 6100 10550 50  0000 C CNN
-F 2 "" H 6100 10700 60  0000 C CNN
-F 3 "" H 6100 10700 60  0000 C CNN
-	1    6100 10700
+P 5250 9800
+F 0 "#PWR032" H 5250 9550 50  0001 C CNN
+F 1 "GND" H 5250 9650 50  0000 C CNN
+F 2 "" H 5250 9800 60  0000 C CNN
+F 3 "" H 5250 9800 60  0000 C CNN
+	1    5250 9800
 	1    0    0    -1
 $EndComp
@@
 	1    13650 6700
 	1    0    0    -1
-$EndComp
-$Comp
-L GND #PWR035
-U 1 1 59242BE2
-P 13650 7600
-F 0 "#PWR035" H 13650 7350 50  0001 C CNN
-F 1 "GND" H 13650 7450 50  0000 C CNN
-F 2 "" H 13650 7600 60  0000 C CNN
-F 3 "" H 13650 7600 60  0000 C CNN
-	1    13650 7600
-	1    0    0    -1
-$EndComp
-$Comp
-L R R23
-U 1 1 59244D3C
-P 13850 7350
-F 0 "R23" V 13930 7350 50  0000 C CNN
-F 1 "10k" V 13850 7350 50  0000 C CNN
-F 2 "project_footprints:R_0402_Hand" V 13780 7350 30  0001 C CNN
-F 3 "" H 13850 7350 30  0000 C CNN
-F 4 "311-10KJRCT-ND" V 13850 7350 60  0001 C CNN "Digikey Part No."
-	1    13850 7350
-	-1   0    0    1
 $EndComp
 $Comp
@@
 $EndComp
 $Comp
-L +3.3V #PWR036
+L +3.3V #PWR035
 U 1 1 59246E04
 P 12100 6700
-F 0 "#PWR036" H 12100 6550 50  0001 C CNN
+F 0 "#PWR035" H 12100 6550 50  0001 C CNN
 F 1 "+3.3V" H 12100 6840 50  0000 C CNN
 F 2 "" H 12100 6700 60  0000 C CNN
@@
 	1    12100 6700
 	1    0    0    -1
-$EndComp
-$Comp
-L GND #PWR037
-U 1 1 59246E0D
-P 12100 7600
-F 0 "#PWR037" H 12100 7350 50  0001 C CNN
-F 1 "GND" H 12100 7450 50  0000 C CNN
-F 2 "" H 12100 7600 60  0000 C CNN
-F 3 "" H 12100 7600 60  0000 C CNN
-	1    12100 7600
-	1    0    0    -1
-$EndComp
-$Comp
-L R R22
-U 1 1 59246E14
-P 12300 7350
-F 0 "R22" V 12380 7350 50  0000 C CNN
-F 1 "10k" V 12300 7350 50  0000 C CNN
-F 2 "project_footprints:R_0402_Hand" V 12230 7350 30  0001 C CNN
-F 3 "" H 12300 7350 30  0000 C CNN
-F 4 "311-10KJRCT-ND" V 12300 7350 60  0001 C CNN "Digikey Part No."
-	1    12300 7350
-	-1   0    0    1
 $EndComp
 $Comp
@@
 HALL2
 $Comp
-L +3.3V #PWR038
+L +3.3V #PWR036
 U 1 1 5925739B
 P 10950 1050
-F 0 "#PWR038" H 10950 900 50  0001 C CNN
+F 0 "#PWR036" H 10950 900 50  0001 C CNN
 F 1 "+3.3V" H 10950 1190 50  0000 C CNN
 F 2 "" H 10950 1050 60  0000 C CNN
@@
 	7400 8650 6900 8650
 Wire Wire Line
-	6600 8650 5950 8650
+	5250 8650 6600 8650
 Wire Wire Line
 	5950 8600 5950 9100
@@
 	6150 9550 6100 9550
 Wire Wire Line
-	6100 9550 6100 9800
+	5250 8650 5250 8900
 Wire Wire Line
 	10100 1700 9750 1700
@@
 	10950 1700 10700 1700
 Wire Wire Line
-	6100 10100 6100 10250
-Wire Wire Line
-	6250 10200 6100 10200
-Connection ~ 6100 10200
-Wire Wire Line
-	6100 10550 6100 10700
-Wire Wire Line
-	13400 6950 13650 6950
-Wire Wire Line
-	13650 6950 13650 6700
-Wire Wire Line
-	13400 7150 13950 7150
+	5250 9200 5250 9350
+Wire Wire Line
+	5400 9300 5250 9300
+Connection ~ 5250 9300
+Wire Wire Line
+	5250 9650 5250 9800
+Wire Wire Line
+	13650 6950 13400 6950
+Wire Wire Line
+	13650 6700 13650 6950
 Wire Wire Line
 	13400 7350 13650 7350
-Wire Wire Line
-	13650 7350 13650 7600
-Wire Wire Line
-	13850 7100 13850 7200
-Connection ~ 13850 7150
 Wire Wire Line
 	13850 6800 13650 6800
 Connection ~ 13650 6800
 Wire Wire Line
-	13850 7500 13850 7550
-Wire Wire Line
-	13850 7550 13650 7550
-Connection ~ 13650 7550
-Wire Wire Line
-	11850 6950 12100 6950
-Wire Wire Line
-	12100 6950 12100 6700
+	12100 6950 11850 6950
+Wire Wire Line
+	12100 6700 12100 6950
 Wire Wire Line
 	11850 7150 12400 7150
-Wire Wire Line
-	11850 7350 12100 7350
-Wire Wire Line
-	12100 7350 12100 7600
-Wire Wire Line
-	12300 7100 12300 7200
 Connection ~ 12300 7150
 Wire Wire Line
@@
 Connection ~ 12100 6800
 Wire Wire Line
-	12300 7500 12300 7550
-Wire Wire Line
-	12300 7550 12100 7550
-Connection ~ 12100 7550
-Wire Wire Line
 	10950 1050 10950 1700
 Connection ~ 10950 1350
@@
 	9750 2150 9750 2050
 $Comp
-L GND #PWR039
+L GND #PWR037
 U 1 1 5925D5CC
 P 9650 2200
-F 0 "#PWR039" H 9650 1950 50  0001 C CNN
+F 0 "#PWR037" H 9650 1950 50  0001 C CNN
 F 1 "GND" H 9650 2050 50  0000 C CNN
 F 2 "" H 9650 2200 60  0000 C CNN
@@
 	10800 3750 10850 3750
 $Comp
-L GND #PWR040
+L GND #PWR038
 U 1 1 5927C794
 P 10850 3750
-F 0 "#PWR040" H 10850 3500 50  0001 C CNN
+F 0 "#PWR038" H 10850 3500 50  0001 C CNN
 F 1 "GND" H 10850 3600 50  0000 C CNN
 F 2 "" H 10850 3750 60  0000 C CNN
@@
 Connection ~ 14750 2450
 $Comp
-L GND #PWR041
+L GND #PWR039
 U 1 1 59252694
 P 14750 4450
-F 0 "#PWR041" H 14750 4200 50  0001 C CNN
+F 0 "#PWR039" H 14750 4200 50  0001 C CNN
 F 1 "GND" H 14750 4300 50  0000 C CNN
 F 2 "" H 14750 4450 60  0000 C CNN
@@
 	1    0    0    -1
 $EndComp
+$Comp
+L LED D6
+U 1 1 5955DFC7
+P 6100 10300
+F 0 "D6" H 6100 10400 50  0000 C CNN
+F 1 "CHRG" H 6100 10200 50  0000 C CNN
+F 2 "idlehands_footprints:Led_0603" H 6100 10300 60  0001 C CNN
+F 3 "" H 6100 10300 60  0000 C CNN
+F 4 "160-1436-1-ND" H 6100 10300 60  0001 C CNN "Digikey Part No."
+	1    6100 10300
+	0    1    1    0
+$EndComp
+$Comp
+L R R14
+U 1 1 5955DFCE
+P 6100 9850
+F 0 "R14" V 6180 9850 50  0000 C CNN
+F 1 "1K" V 6100 9850 50  0000 C CNN
+F 2 "project_footprints:R_0402_Hand" V 6030 9850 30  0001 C CNN
+F 3 "" H 6100 9850 30  0000 C CNN
+F 4 "311-1.0KJRCT-ND" V 6100 9850 60  0001 C CNN "Digikey Part No."
+	1    6100 9850
+	1    0    0    -1
+$EndComp
+Wire Wire Line
+	6100 10000 6100 10100
+Wire Wire Line
+	6100 9550 6100 9700
+Wire Wire Line
+	6100 10500 6100 10600
+$Comp
+L VCC #PWR040
+U 1 1 595611F9
+P 5800 10500
+F 0 "#PWR040" H 5800 10350 50  0001 C CNN
+F 1 "VCC" H 5800 10650 50  0000 C CNN
+F 2 "" H 5800 10500 60  0000 C CNN
+F 3 "" H 5800 10500 60  0000 C CNN
+	1    5800 10500
+	1    0    0    -1
+$EndComp
+Wire Wire Line
+	6100 10600 5800 10600
+Wire Wire Line
+	5800 10600 5800 10500
+$Comp
+L 2N7002 Q2
+U 1 1 59572720
+P 12600 8000
+F 0 "Q2" H 12800 8075 50  0000 L CNN
+F 1 "2N7002" H 12800 8000 50  0000 L CNN
+F 2 "TO_SOT_Packages_SMD:SOT-23" H 12800 7925 50  0001 L CIN
+F 3 "" H 12600 8000 50  0000 L CNN
+F 4 "1727-4793-1-ND" H 12600 8000 60  0001 C CNN "Digikey Part No."
+	1    12600 8000
+	1    0    0    -1
+$EndComp
+Wire Wire Line
+	12700 8200 12700 8350
+$Comp
+L GND #PWR041
+U 1 1 59576997
+P 12700 8350
+F 0 "#PWR041" H 12700 8100 50  0001 C CNN
+F 1 "GND" H 12700 8200 50  0000 C CNN
+F 2 "" H 12700 8350 60  0000 C CNN
+F 3 "" H 12700 8350 60  0000 C CNN
+	1    12700 8350
+	1    0    0    -1
+$EndComp
+Wire Wire Line
+	12200 8050 12400 8050
+Wire Wire Line
+	12300 8050 12300 8150
+Connection ~ 12300 8050
+$Comp
+L R_Small R13
+U 1 1 595798D8
+P 12300 8250
+F 0 "R13" H 12330 8270 50  0000 L CNN
+F 1 "100k" H 12330 8210 50  0001 L CNN
+F 2 "project_footprints:R_0402_Hand" H 12300 8250 60  0001 C CNN
+F 3 "" H 12300 8250 60  0000 C CNN
+F 4 "311-100KLRCT-ND" H 12300 8250 60  0001 C CNN "Digikey Part No."
+	1    12300 8250
+	1    0    0    -1
+$EndComp
+$Comp
+L GND #PWR042
+U 1 1 5957B69B
+P 12300 8400
+F 0 "#PWR042" H 12300 8150 50  0001 C CNN
+F 1 "GND" H 12300 8250 50  0000 C CNN
+F 2 "" H 12300 8400 60  0000 C CNN
+F 3 "" H 12300 8400 60  0000 C CNN
+	1    12300 8400
+	1    0    0    -1
+$EndComp
+Wire Wire Line
+	12300 8400 12300 8350
+Wire Wire Line
+	12700 7550 12700 7800
+Text GLabel 12200 8050 0    60   Input ~ 0
+HALLSW
+Wire Wire Line
+	12300 7150 12300 7100
+Connection ~ 12700 7550
+Wire Wire Line
+	11850 7350 12100 7350
+Wire Wire Line
+	12100 7350 12100 7550
+Wire Wire Line
+	12100 7550 13650 7550
+Wire Wire Line
+	13650 7550 13650 7350
+Wire Wire Line
+	13400 7150 13950 7150
+Wire Wire Line
+	13850 7100 13850 7150
+Connection ~ 13850 7150
+Text GLabel 6250 2450 2    60   Input ~ 0
+HALLSW
 $EndSCHEMATC
